Commit message: fix damping and friction coefs and add color args

File: urdf/include/addon_macro.urdf.xacro (robot description, xacro)
@@ -49,6 +49,6 @@
       <axis xyz="0 0 0" />
     </joint>
-    <gazebo reference="${addon}">
-      <material>Gazebo/Black</material>
+    <gazebo reference="${addon}_link">
+      <material>${base_prop[addon]['color']}</material>
     </gazebo>
   </xacro:macro>

File: urdf/include/common_macros.urdf.xacro (robot description, xacro)
@@ -60,5 +60,5 @@
     </link>
     <gazebo reference="${prefix}_wheel">
-      <material>Gazebo/Grey</material>
+      <material>Gazebo/FlatBlack</material>
     </gazebo>
     <joint name="${prefix}_wheel_joint" type="continuous">
@@ -142,5 +142,5 @@
     </joint>
     <gazebo reference="${prefix}_motor">
-      <material>Gazebo/SkyBlue</material>
+      <material>${motor_props['color']}</material>
       <turnGravityOff>false</turnGravityOff>
     </gazebo>

File: urdf/include/remo_base_macro.urdf.xacro (robot description, xacro)
@@ -50,4 +50,7 @@
     </collision>
     </link>
+    <gazebo reference="base_link">
+      <material>Gazebo/Grey</material>
+    </gazebo>
   </xacro:macro>
 </robot>

File: urdf/include/remo_caster_macro.urdf.xacro (robot description, xacro)
@@ -61,5 +61,5 @@
     </joint>
     <gazebo reference="${prefix}_caster_base_link">
-      <material>Gazebo/Black</material>
+      <material>Gazebo/Grey</material>
     </gazebo>
     <!-- caster hub -->
@@ -109,5 +109,5 @@
     </joint>
     <gazebo reference="${prefix}_caster_rotation_link">
-      <material>Gazebo/Black</material>
+      <material>Gazebo/Grey</material>
     </gazebo>
     <!-- caster wheel -->
@@ -153,5 +153,6 @@
       <child link="${prefix}_caster_wheel_link" />
       <axis xyz="0 1 0" />
-      <dynamics damping="0.01" friction="0.0"/>
+      <!-- Don't turn damping higher than 0.001, otherwise caster and wheels merge in simulation (bug?) -->
+      <dynamics damping="0.001" friction="0.0"/>
     </joint>
     <gazebo reference="${prefix}_caster_wheel_link">

File: urdf/include/robot.gazebo.xacro (robot description, xacro)
@@ -25,4 +25,6 @@
     </gazebo>
   </xacro:macro>
+  <!-- http://gazebosim.org/tutorials?tut=friction -->
+  <!-- http://sdformat.org/spec?ver=1.5&elem=collision#ode_mu -->
   <!-- https://answers.ros.org/question/231880/how-to-improve-amcl-pose-estimate/ -->
   <!-- https://answers.ros.org/question/30539/choosing-the-right-coefficients-for-gazebo-simulation/ -->
@@ -33,30 +35,30 @@
     <!--xacro:set_wheel_friction link="rear_caster_wheel_link" friction="${friction}"/-->
     <gazebo reference="front_right_wheel">
-      <mu1>20</mu1>
-      <mu2>10</mu2>
-      <kp>10000000000.0</kp>
-      <kd>0.001</kd>
-      <minDepth>0.001</minDepth>
-      <maxVel>0.1</maxVel>
-      <fdir1>1 0 0</fdir1>
+      <mu1>200</mu1>                <!-- Coefficient of friction in the range of [0..1] (default 1) (docs seems wrong increasing to 200 improves behaviour) -->
+      <mu2>200</mu2>                <!-- Second coefficient of friction in the range of [0..1] (default 1) (docs seems wrong increasing to 200 improves behaviour)-->
+      <kp>1000000000000</kp>      <!-- dynamically "stiffness"-equivalent coefficient for contact joints (default 1000000000000)-->
+      <kd>0</kd>                  <!-- dynamically "damping"-equivalent coefficient for contact joints (default 1) -->
+      <minDepth>0.01</minDepth>      <!-- minimum allowable depth before contact correction impulse is applied (default 0) -->
+      <maxVel>0.01</maxVel> <!-- maximum contact correction velocity truncation term (default 0.01)-->
+      <fdir1>0 0 1</fdir1>   <!-- 3-tuple specifying direction of mu1 in the collision local reference frame (default 0 0 0) -->
       <material>Gazebo/FlatBlack</material>
     </gazebo>
     <gazebo reference="front_left_wheel">
-      <mu1>20</mu1>
-      <mu2>10</mu2>
-      <kp>1000000000.0</kp>
-      <kd>0.001</kd>
-      <minDepth>0.001</minDepth>
-      <maxVel>0.1</maxVel>
-      <fdir1>1 0 0</fdir1>
+      <mu1>200</mu1>
+      <mu2>200</mu2>
+      <kp>1000000000000</kp>
+      <kd>0</kd>
+      <minDepth>0.01</minDepth>
+      <maxVel>0.01</maxVel>
+      <fdir1>0 0 1</fdir1>
       <material>Gazebo/FlatBlack</material>
     </gazebo>
     <gazebo reference="rear_caster_rotation_link">
-      <mu1>0.001</mu1>
-      <mu2>0.001</mu2>
-      <kp>1000000000.0</kp>
-      <kd>0.001</kd>
-      <minDepth>0.001</minDepth>
-      <maxVel>1.0</maxVel>
+      <mu1>0.01</mu1>
+      <mu2>0.01</mu2>
+      <kp>1000000000000</kp>
+      <kd>0</kd>
+      <minDepth>0.0</minDepth>
+      <!-- maxVel>1.0</maxVel-->
       <!--fdir1>0 0 1</fdir1-->
       <material>Gazebo/FlatBlack</material>
@@ -65,9 +67,9 @@
       <mu1>0.01</mu1>
       <mu2>0.01</mu2>
-      <kp>1000000000.0</kp>
-      <kd>0.001</kd>
-      <minDepth>0.001</minDepth>
-      <maxVel>1.0</maxVel>
-      <material>Gazebo/FlatBlack</material>
+      <kp>1000000000000</kp>
+      <kd>0</kd>
+      <minDepth>0.01</minDepth>
+      <!-- maxVel>10.0</maxVel -->
+      <material>Gazebo/White</material>
     </gazebo>
   </xacro:macro>
